Commit message: feat: update urdf and wheel damping

File: assets/robots/roller_skating_robot.urdf (robot description, URDF)
Before this commit: robot roller_skating_robot, 21 links, 20 joints
Links:
- link base_link: mass 3.0 -> 30.0
- link left_foot: mass 0.7 -> 1.0
- link left_shank: mass 0.8 -> 3.0
- link left_thigh: mass 1.0 -> 6.0
- link right_foot: mass 0.7 -> 1.0
- link right_shank: mass 0.8 -> 3.0
- link right_thigh: mass 1.0 -> 6.0
Joints:
- joint left_ankle_pitch_joint: limit lower=-0.5236 upper=0.5236 effort=50 velocity=3.0 -> lower=-0.5236 upper=0.5236 effort=100 velocity=3.0
- joint left_ankle_roll_joint: axis 1 0 0 -> (none); limit lower=-0.2618 upper=0.2618 effort=50 velocity=3.0 -> (none); type revolute -> fixed
- joint left_hip_pitch_joint: limit lower=-1.2 upper=1.2 effort=50 velocity=3.0 -> lower=-1.2 upper=1.2 effort=100 velocity=3.0
- joint left_hip_roll_joint: limit lower=-0.7854 upper=0.7854 effort=50 velocity=3.0 -> lower=-0.7854 upper=0.7854 effort=100 velocity=3.0
- joint left_hip_yaw_joint: limit lower=-1.0 upper=1.0 effort=50 velocity=3.0 -> lower=-1.0 upper=1.0 effort=100 velocity=3.0
- joint left_knee_joint: limit lower=0 upper=2.0 effort=50 velocity=3.0 -> lower=0 upper=2.0 effort=100 velocity=3.0
- joint right_ankle_pitch_joint: limit lower=-0.5236 upper=0.5236 effort=50 velocity=3.0 -> lower=-0.5236 upper=0.5236 effort=100 velocity=3.0
- joint right_ankle_roll_joint: axis 1 0 0 -> (none); limit lower=-0.2618 upper=0.2618 effort=50 velocity=3.0 -> (none); type revolute -> fixed
- joint right_hip_pitch_joint: limit lower=-1.2 upper=1.2 effort=50 velocity=3.0 -> lower=-1.2 upper=1.2 effort=100 velocity=3.0
- joint right_hip_roll_joint: limit lower=-0.7854 upper=0.7854 effort=50 velocity=3.0 -> lower=-0.7854 upper=0.7854 effort=100 velocity=3.0
- joint right_hip_yaw_joint: limit lower=-1.0 upper=1.0 effort=50 velocity=3.0 -> lower=-1.0 upper=1.0 effort=100 velocity=3.0
- joint right_knee_joint: limit lower=0 upper=2.0 effort=50 velocity=3.0 -> lower=0 upper=2.0 effort=100 velocity=3.0

Commit message: feat: medium weight robot and param

File: assets/robots/roller_skating_robot.urdf (robot description, URDF)
Before this commit: robot roller_skating_robot, 21 links, 20 joints
Links:
- link base_link: mass 30.0 -> 6.0
- link left_foot: mass 1.0 -> 0.7
- link left_shank: mass 3.0 -> 0.8
- link left_thigh: mass 6.0 -> 1.0
- link right_foot: mass 1.0 -> 0.7
- link right_shank: mass 3.0 -> 0.8
- link right_thigh: mass 6.0 -> 1.0
Joints:
- joint left_ankle_pitch_joint: limit lower=-0.5236 upper=0.5236 effort=100 velocity=3.0 -> lower=-0.5236 upper=0.5236 effort=50 velocity=3.0
- joint left_hip_pitch_joint: limit lower=-1.2 upper=1.2 effort=100 velocity=3.0 -> lower=-1.2 upper=1.2 effort=50 velocity=3.0
- joint left_hip_roll_joint: limit lower=-0.7854 upper=0.7854 effort=100 velocity=3.0 -> lower=-0.7854 upper=0.7854 effort=50 velocity=3.0
- joint left_hip_yaw_joint: limit lower=-1.0 upper=1.0 effort=100 velocity=3.0 -> lower=-1.0 upper=1.0 effort=50 velocity=3.0
- joint left_knee_joint: limit lower=0 upper=2.0 effort=100 velocity=3.0 -> lower=0 upper=2.0 effort=50 velocity=3.0
- joint right_ankle_pitch_joint: limit lower=-0.5236 upper=0.5236 effort=100 velocity=3.0 -> lower=-0.5236 upper=0.5236 effort=50 velocity=3.0
- joint right_hip_pitch_joint: limit lower=-1.2 upper=1.2 effort=100 velocity=3.0 -> lower=-1.2 upper=1.2 effort=50 velocity=3.0
- joint right_hip_roll_joint: limit lower=-0.7854 upper=0.7854 effort=100 velocity=3.0 -> lower=-0.7854 upper=0.7854 effort=50 velocity=3.0
- joint right_hip_yaw_joint: limit lower=-1.0 upper=1.0 effort=100 velocity=3.0 -> lower=-1.0 upper=1.0 effort=50 velocity=3.0
- joint right_knee_joint: limit lower=0 upper=2.0 effort=100 velocity=3.0 -> lower=0 upper=2.0 effort=50 velocity=3.0
